File: IMU9.brd (EAGLE design)
At the start: 20.3 x 12.7 mm, 22 parts, among them IC1 MCP1700T-3302E/TT, Q1 RJU003N03 N-MOSFET, Q2 RJU003N03 N-MOSFET

Commit message: Added Adelmo Eloy as designer Added notes to schematic about max parameters Improved silkscreen Improved designator positions Improved part designators and values
Parts:
- H1: value M01PTH -> GND
- H2: value M01PTH -> SDA
- H3: value M01PTH -> SCL
- H4: value M01PTH -> VCC
- H5: value M01PTH -> INT
- R1, R2: value 10K 0402 -> 4K7 0402
- renumbered GND to H1, INT to H5, SCL to H3, SDA to H2, U$1 to IC2, VCC to H4
Other:
- board text added: "(c) 2014 Freetronics"
- board text added: "2.75-6V"
- board text removed: "(c) 2013 Freetronics"
- board text removed: "2.3-6V"

Commit message: Bridged across I2C pull-up cut track jumpers Shortened URL
Routing:
- net N$15: track 0.00 -> 0.51 mm
- net N$13: track 0.00 -> 0.51 mm
Other:
- board text added: "tron.cc/imu9"
- board text added: "v1.1"
- board text removed: "freetronics.com/imu9"
- board text removed: "v1.0"
Changed lines of the file:
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@@
 <?xml version="1.0" encoding="utf-8"?>
 <!DOCTYPE eagle SYSTEM "eagle.dtd">
-<eagle version="6.3">
+<eagle version="6.5.0">
 <drawing>
 <settings>
@@
 <wire x1="14.224" y1="4.572" x2="15.24" y2="5.588" width="0.254" layer="22" curve="90.022562"/>
 <wire x1="15.24" y1="5.588" x2="14.351" y2="6.604" width="0.254" layer="22" curve="89.988722"/>
-<text x="16.129" y="7.62" size="0.8636" layer="22" font="vector" ratio="16" rot="MR0">freetronics.com/imu9</text>
+<text x="16.129" y="7.112" size="1.27" layer="22" font="vector" ratio="16" rot="MR0">tron.cc/imu9</text>
 <text x="2.794" y="0.762" size="0.8636" layer="22" font="vector" ratio="18" rot="MR90">SKU: IMU9</text>
 <text x="14.605" y="5.207" size="1.016" layer="22" font="vector" ratio="15" rot="MR0">freetronics</text>
@@
 <text x="15.2908" y="2.286" size="1.524" layer="21" font="vector" ratio="15">IMU9</text>
 <circle x="9.525" y="9.017" radius="0.254" width="0.254" layer="21"/>
-<text x="16.002" y="1.778" size="1.016" layer="22" ratio="15" rot="MR180">v1.0</text>
+<text x="16.002" y="1.778" size="1.016" layer="22" ratio="15" rot="MR180">v1.1</text>
 <text x="0.762" y="7.5946" size="0.8128" layer="21" ratio="15">AD0</text>
 <text x="8.636" y="12.3952" size="0.8128" layer="21" font="vector" ratio="15" rot="R270">INT</text>
@@
 <signal name="N$12">
 </signal>
+<signal name="N$13">
+<wire x1="19.05" y1="6.858" x2="19.05" y2="6.35" width="0.2032" layer="16"/>
+</signal>
+<signal name="N$15">
+<wire x1="19.05" y1="5.334" x2="19.05" y2="4.826" width="0.2032" layer="16"/>
+</signal>
 </signals>
+<errors>
+</errors>
 </board>
 </drawing>
